File: pcb/nearness.sch (KiCad schematic (older format))
At the start: 52 parts, among them J1 PJ301M12, J2 PJ301M12, J3 PJ301M12, J4 PJ301M12, J5 PJ301M12, J6 PJ301M12, J7 PJ301M12, J8 PJ301M12, J9 PJ301M12, P1 CONN_01X05, P2 CONN_01X05, P3 CONN_01X05, P4 CONN_01X05, P5 CONN_01X03, P6 CONN_01X03, P7 CONN_01X03, U1 LME49720, U2 LME49720

Commit message: Upgrade project to KiCad 5
Upgrade project, library, schematic, and PCB files to KiCad 5. Remap
symbols to the Device and Connector libraries, using different symbols
for male and female pin headers. Re-annotate schematic. Re-fill zones.
Ignore KiCad 5 backup and cache files.
Parts:
- C1, C2, C3, C4, C5, C6, C7, C8: symbol C -> Device:C
- D1, D2: symbol D -> Device:D
- J1, J2, J3, J4, J5, J6, J7, J8, J9: symbol PJ301M12 -> pj301m12:PJ301M12
- P1, P2: symbol CONN_01X05 -> Connector:Conn_01x05_Female
- P3, P4: symbol CONN_01X05 -> Connector:Conn_01x05_Male
- P5, P6, P7: symbol CONN_01X03 -> Connector:Conn_01x03_Male
- R1, R10, R11, R12, R13, R14, R15, R16, R17, R18, R19, R2, R20, R21, R22, R23, R24, R3, R4, R5, R6, R7, R8, R9: symbol R -> Device:R
- U1, U2: symbol LME49720 -> lme49720:LME49720
